File: CameraTriggerR2PCB/CameraIO.sch (KiCad schematic (older format))
At the start: 13 parts, among them J1 Camera 3.5mm, J2 Camera 2.5mm, Q1 PN2222A, Q2 PN2222A, U1 ILD74, U2 ILD74

Commit message: Add files via upload
First cut at modules
Other:
- note added: "TODO - put two sets of jacks on each"

Commit message: Add files via upload
Changes from 5/17 Zoom sensor
Parts:
- added J12: Camera 2.5mm, CameraTriggerPCB:CUI_SJ1-2503A, symbol Connector:AudioJack3
- added J13: Camera 3.5mm, Connector_Audio:Jack_3.5mm_CUI_SJ1-3533NG_Horizontal_CircularHoles, symbol Connector:AudioJack3
Connections:
- wire segments 62 -> 79
- no-connect marks 2 -> 0
Other:
- note removed: "TODO - put two sets of jacks on each"
