File: CameraTriggerR2PCB/CameraTrigger.sch (KiCad schematic (older format))
At the start: 57 parts, among them J1 Power, J10 feather short, J11 Ada2633, J12 Camera 2.5mm, J13 +5V Always on, J14 Ext power switch, J2 Camera 3.5mm, J3 Aux out, J4 HighLowIn, J5 Laser, J6 Sensor, J7 Trig, J8 Arm, J9 Ada3178, Q1 PN2222A, Q2 PN2222A, Q3 PN2222A, SW1 SW_Power, SW2 SW_Trigger, SW3 SW_Poll, SW4 SW_Arm, U1 LM7805_TO220, U2 ILD74, U3 ILD74

Commit message: Moved jacks closer to board edge
Parts:
- removed H5: MountingHole, MountingHole:MountingHole_4.5mm, symbol Mechanical:MountingHole
- removed J10: feather short, Connector_PinHeader_2.54mm:PinHeader_1x12_P2.54mm_Vertical, symbol Connector_Generic:Conn_01x12
- removed J9: Ada3178, Connector_PinHeader_2.54mm:PinHeader_1x16_P2.54mm_Vertical, symbol Connector_Generic:Conn_01x16
- removed SW1: SW_Power, Button_Switch_THT:SW_DIP_SPSTx01_Slide_6.7x4.1mm_W7.62mm_P2.54mm_LowProfile, symbol Switch:SW_SPST
- added C5, C6: 0.01 μF, Capacitor_THT:C_Disc_D7.5mm_W2.5mm_P5.00mm, symbol Device:C
- added IC1: 3178, 3178, symbol SamacSys_Parts:3178
- added SW1: AS11CB, CameraTriggerPCB:AS11CB, symbol SamacSys_Parts:AS11CB
- added TP1: TestPoint, TestPoint:TestPoint_Keystone_5000-5004_Miniature, symbol Connector:TestPoint
Connections:
- wire segments 225 -> 235
- no-connect marks 11 -> 17
Other:
- moved on the sheet: D5, GND1, J13

Commit message: Add files via upload
Broke schematic into hierarchical sheets
Parts:
- removed BZ1: Buzzer, Buzzer_Beeper:Buzzer_TDK_PS1240P02BT_D12.2mm_H6.5mm, symbol Device:Buzzer
- removed C1: 25uf, Capacitor_THT:CP_Radial_Tantal_D5.0mm_P5.00mm, symbol Device:CP
- removed C2: 0.1uf, Capacitor_THT:CP_Radial_Tantal_D5.0mm_P5.00mm, symbol Device:C
- removed C3, C4, C5, C6: 0.01 μF, Capacitor_THT:C_Disc_D7.5mm_W2.5mm_P5.00mm, symbol Device:C
- removed D1: LED Arm, LED_THT:LED_D3.0mm, symbol Device:LED
- removed D2: LED Trig, LED_THT:LED_D3.0mm, symbol Device:LED
- removed D3: D, Diode_THT:D_DO-201AD_P12.70mm_Horizontal, symbol Device:D
- removed D4: PWR, LED_THT:LED_D3.0mm, symbol Device:LED
- removed D5: LED Focus, LED_THT:LED_D3.0mm, symbol Device:LED
- removed GND1, TP1: TestPoint, TestPoint:TestPoint_Keystone_5000-5004_Miniature, symbol Connector:TestPoint
- removed H1, H4: (no value), MountingHole:MountingHole_3.7mm_Pad, symbol Mechanical:MountingHole_Pad
- removed H2, H3: MountingHole_Pad, MountingHole:MountingHole_3.7mm_Pad, symbol Mechanical:MountingHole_Pad
- removed IC1: 3178, 3178, symbol SamacSys_Parts:3178
- removed J1: Power, Connector_AMASS:AMASS_XT30U-F_1x02_P5.0mm_Vertical, symbol Connector:Screw_Terminal_01x02
- removed J11: Ada2633, Connector_PinHeader_2.54mm:PinHeader_1x09_P2.54mm_Vertical, symbol Connector:Conn_01x09_Female
- removed J12: Camera 2.5mm, CameraTriggerPCB:CUI_SJ1-2503A, symbol Connector:AudioJack3
- removed J13: +5V Always on, TerminalBlock_TE-Connectivity:TerminalBlock_TE_282834-2_1x02_P2.54mm_Horizontal, symbol Connector:Screw_Terminal_01x02
- removed J14: Ext power switch, TerminalBlock_TE-Connectivity:TerminalBlock_TE_282834-2_1x02_P2.54mm_Horizontal, symbol Connector:Screw_Terminal_01x02
- removed J2: Camera 3.5mm, Connector_Audio:Jack_3.5mm_CUI_SJ1-3533NG_Horizontal_CircularHoles, symbol Connector:AudioJack3
- removed J3: Aux out, TerminalBlock_TE-Connectivity:TerminalBlock_TE_282834-2_1x02_P2.54mm_Horizontal, symbol Connector:Screw_Terminal_01x02
- removed J4: HighLowIn, TerminalBlock_TE-Connectivity:TerminalBlock_TE_282834-3_1x03_P2.54mm_Horizontal, symbol Connector:Screw_Terminal_01x03
- removed J5: Laser, TerminalBlock_TE-Connectivity:TerminalBlock_TE_282834-2_1x02_P2.54mm_Horizontal, symbol Connector:Screw_Terminal_01x02
- removed J6: Sensor, TerminalBlock_TE-Connectivity:TerminalBlock_TE_282834-3_1x03_P2.54mm_Horizontal, symbol Connector:Screw_Terminal_01x03
- removed J7: Trig, TerminalBlock_TE-Connectivity:TerminalBlock_TE_282834-2_1x02_P2.54mm_Horizontal, symbol Connector:Screw_Terminal_01x02
- removed J8: Arm, TerminalBlock_TE-Connectivity:TerminalBlock_TE_282834-2_1x02_P2.54mm_Horizontal, symbol Connector:Screw_Terminal_01x02
- removed Q1, Q2, Q3: PN2222A, Package_TO_SOT_THT:TO-92_Inline, symbol Transistor_BJT:PN2222A
- removed R1, R2, R5: 1K, Resistor_THT:R_Axial_DIN0207_L6.3mm_D2.5mm_P7.62mm_Horizontal, symbol Device:R
- removed R3: 5K, Resistor_THT:R_Axial_DIN0207_L6.3mm_D2.5mm_P7.62mm_Horizontal, symbol Device:R
- removed R4: 220, Resistor_THT:R_Axial_DIN0207_L6.3mm_D2.5mm_P7.62mm_Horizontal, symbol Device:R
- removed R6, R7: 50, Resistor_THT:R_Axial_DIN0207_L6.3mm_D2.5mm_P7.62mm_Horizontal, symbol Device:R
- removed R8: 15K, Resistor_THT:R_Axial_DIN0207_L6.3mm_D2.5mm_P7.62mm_Horizontal, symbol Device:R
- removed SW1: AS11CB, CameraTriggerPCB:AS11CB, symbol SamacSys_Parts:AS11CB
- removed SW2: SW_Trigger, Button_Switch_THT:KSA_Tactile_SPST, symbol Switch:SW_Push
- removed SW3: SW_Poll, Button_Switch_THT:KSA_Tactile_SPST, symbol Switch:SW_Push
- removed SW4: SW_Arm, Button_Switch_THT:KSA_Tactile_SPST, symbol Switch:SW_Push
- removed TP1+5: +5V, TestPoint:TestPoint_Keystone_5010-5014_Multipurpose, symbol Connector:TestPoint
- removed TP2+3.3V1: +3.3V, TestPoint:TestPoint_Keystone_5010-5014_Multipurpose, symbol Connector:TestPoint
- removed TP3Arm1, TP6Arm1: Arm, TestPoint:TestPoint_Keystone_5010-5014_Multipurpose, symbol Connector:TestPoint
- removed TP4Fire1: Fire, TestPoint:TestPoint_Keystone_5010-5014_Multipurpose, symbol Connector:TestPoint
- removed TP5Trigger1: Trigger, TestPoint:TestPoint_Keystone_5010-5014_Multipurpose, symbol Connector:TestPoint
- removed TP7Poll1: Poll, TestPoint:TestPoint_Keystone_5010-5014_Multipurpose, symbol Connector:TestPoint
- removed TP8: HighLowIn, TestPoint:TestPoint_Keystone_5010-5014_Multipurpose, symbol Connector:TestPoint
- removed TP9: LowHighIn, TestPoint:TestPoint_Keystone_5010-5014_Multipurpose, symbol Connector:TestPoint
- removed U1: LM7805_TO220, Package_TO_SOT_THT:TO-220-3_Vertical, symbol Regulator_Linear:LM7805_TO220
- removed U2, U3: ILD74, Package_DIP:DIP-8_W7.62mm, symbol Isolator:ILD74
Connections:
- net labels removed: +3.3V, +5V, +7.5V, 13, A0, A1, A2, A3, A4, A5, AREF, Adafruit3178, ArmIn, ArmInd, AuxIn, AuxOut, Buzzer, CS, EN, FREE, Focus, GND, IRQ, MISO, MOSI, PbTrigIn, Poll, RX, SCK, SCL, SDA, SensorIn, Shutter, TX, VBAT, VUSB, ~RST
- wire segments 235 -> 0
- no-connect marks 17 -> 0
Other:
- note removed: "+3.3V"
- note removed: "+3v"
- note removed: "0"
- note removed: "1"
- note removed: "10"
- note removed: "11"
- note removed: "12"
- note removed: "14"
- note removed: "15"
- note removed: "16"
- note removed: "17"
- note removed: "18"
- note removed: "19"
- note removed: "20"
- note removed: "21"
- note removed: "22"
- note removed: "23"
- note removed: "24"
- note removed: "5"
- note removed: "6"
- note removed: "9"
- note removed: "GND"

Commit message: Add files via upload
First cut at modules
Changed lines of the file:
@@
 $Descr A4 11693 8268
 encoding utf-8
-Sheet 1 8
+Sheet 1 9
 Title ""
 Date ""
@@
 RocketTrig  Curtis Heisey
 $Sheet
-S 5500 1500 1950 1450
+S 5400 1250 1950 1450
 U 5EBC562C
 F0 "CameraIO" 50
 F1 "CameraIO.sch" 50
-F2 "Shutter" I L 5500 1850 50
-F3 "Focus" I L 5500 2000 50
+F2 "Shutter" I L 5400 1600 50
+F3 "Focus" I L 5400 1750 50
 $EndSheet
 $Sheet
@@
 $EndSheet
 $Sheet
-S 2100 4350 950  550
-U 5ECB0F2B
-F0 "AdafruitBT" 50
-F1 "AdafruitBT.sch" 50
-F2 "IRQ" I L 2100 4450 50
-F3 "CS" I L 2100 4550 50
-F4 "MOSI" I L 2100 4650 50
-F5 "MISO" I L 2100 4800 50
-F6 "SCK" I R 3050 4500 50
-$EndSheet
-$Sheet
-S 4150 2550 1150 3500
-U 5ECB134F
-F0 "MCU LoRa" 50
-F1 "MCU LoRa.sch" 50
-F2 "PbTrigIn" I L 4150 2900 50
-F3 "ArmIn" I L 4150 3050 50
-F4 "Poll" I L 4150 3200 50
-F5 "AuxIn" I L 4150 3450 50
-F6 "IRQ" I L 4150 3700 50
-F7 "CS" I L 4150 3850 50
-F8 "SCK" I L 4150 4000 50
-F9 "MOSI" I L 4150 4150 50
-F10 "MISO" I L 4150 4300 50
-F11 "Shutter" I L 4150 4400 50
-F12 "Focus" I L 4150 4550 50
-F13 "Buzzer" I L 4150 4750 50
-F14 "AuxOut" I L 4150 4900 50
-F15 "ArmInd" I L 4150 5000 50
-F16 "SensorIn" I L 4150 5150 50
-$EndSheet
-$Sheet
 S 2200 3200 1050 700
 U 5ECC61B0
@@
 F2 "Buzzer" I L 2200 3450 50
 $EndSheet
+$Sheet
+S 8200 3850 1650 1200
+U 5EBC71CE
+F0 "RFM95" 50
+F1 "RFM95.sch" 50
+F2 "RFM95_SCK" I L 8200 4200 50
+F3 "RFM95_MOSI" I L 8200 4400 50
+F4 "RFM95_MISO" I L 8200 4550 50
+F5 "RFM95_CS" I L 8200 4650 50
+F6 "RFM95_RESET" I L 8200 4750 50
+F7 "RFM95_IRQ" I L 8200 4850 50
+$EndSheet
+$Sheet
+S 9200 2000 1550 1300
+U 5EBC729C
+F0 "WiFi_BT" 50
+F1 "WiFi_BT.sch" 50
+$EndSheet
+$Sheet
+S 4150 2450 900  1500
+U 5EBF5198
+F0 "MCU64pin" 50
+F1 "MCU64pin.sch" 50
+$EndSheet
 $EndSCHEMATC

Commit message: Add files via upload
Changes from 5/17 Zoom sensor
Changed lines of the file:
@@
 F0 "Power" 50
 F1 "Power.sch" 50
+F2 "V_bat_monitor" I L 1800 1250 50
 $EndSheet
 $Sheet
@@
 F0 "WiFi_BT" 50
 F1 "WiFi_BT.sch" 50
+F2 "BT_WIFI_TX" I L 9200 2200 50
+F3 "BT_WIFI_RX" I L 9200 2300 50
+F4 "BT_WIFI_RTS" I L 9200 2400 50
+F5 "BT_WIFI_CTS" I L 9200 2550 50
+F6 "Reset_N" I L 9200 2700 50
 $EndSheet
 $Sheet
-S 4150 2450 900  1500
+S 4150 2450 1200 2300
 U 5EBF5198
 F0 "MCU64pin" 50
 F1 "MCU64pin.sch" 50
+F2 "RFM95_SCK" I L 4150 2550 50
+F3 "RFM95_CS" I L 4150 2600 50
+F4 "RFM95_RESET" I L 4150 2650 50
+F5 "RFM95_IRQ" I L 4150 2700 50
+F6 "BT_WIFI_MISO" I L 4150 2750 50
+F7 "BT_WIFI_MOSI" I L 4150 2850 50
+F8 "BT_WIFI_CS" I L 4150 2950 50
+F9 "BT_WIFI_SCK" I L 4150 3050 50
+F10 "SensorIn" I L 4150 3150 50
+F11 "ArmInd" I L 4150 3200 50
+F12 "AuxIn" I L 4150 3250 50
+F13 "AuxOut" I L 4150 3300 50
+F14 "Buzzer" I L 4150 3350 50
+F15 "Camera" I L 4150 3450 50
+F16 "PbTrigIn" I L 4150 3600 50
+F17 "ArmIn" I L 4150 3550 50
+F18 "Poll" I L 4150 3800 50
+F19 "V_bat_monitor" I L 4150 3700 50
+F20 "RFM95_MISO" I R 5350 2750 50
+F21 "RFM95_MOSI" I R 5350 2850 50
 $EndSheet
 $EndSCHEMATC
