File: CameraTriggerR2PCB/Power.sch (KiCad schematic (older format))
At the start: 16 parts, among them J3 +5V Always on, J4 Ext power switch, J5 Power, SW1 AS11CB, U3 LM7805_TO220

Commit message: Add files via upload
First cut at modules
Parts:
- added C?: 25uf, Capacitor_THT:CP_Radial_Tantal_D5.0mm_P5.00mm, symbol Device:CP
- added C?: 0.1uf, Capacitor_THT:CP_Radial_Tantal_D5.0mm_P5.00mm, symbol Device:C
- added R? (x2): R, symbol Device:R
- added U?: LM7803_TO220, Package_TO_SOT_THT:TO-220-3_Vertical, symbol Regulator_Linear:LM7805_TO220
Connections:
- net labels added: +3.3V, V_bat_monitor
- wire segments 44 -> 56

Commit message: Add files via upload
Changes from 5/17 Zoom sensor
Parts:
- gave numbers to parts that had none: 5
Changed lines of the file:
@@
 P 4450 5700
 AR Path="/5EBF8C68" Ref="#FLG?"  Part="1"
-AR Path="/5EBC5EC2/5EBF8C68" Ref="#FLG?"  Part="1"
-F 0 "#FLG?" H 4450 5775 50  0001 C CNN
+AR Path="/5EBC5EC2/5EBF8C68" Ref="#FLG04"  Part="1"
+F 0 "#FLG04" H 4450 5775 50  0001 C CNN
 F 1 "PWR_FLAG" H 4450 5873 50  0000 C CNN
 F 2 "" H 4450 5700 50  0001 C CNN
@@
 P 3900 5700
 AR Path="/5EBF8C75" Ref="U?"  Part="1"
-AR Path="/5EBC5EC2/5EBF8C75" Ref="U?"  Part="1"
-F 0 "U?" H 3900 5942 50  0000 C CNN
+AR Path="/5EBC5EC2/5EBF8C75" Ref="U4"  Part="1"
+F 0 "U4" H 3900 5942 50  0000 C CNN
 F 1 "LM7803_TO220" H 3900 5851 50  0000 C CNN
 F 2 "Package_TO_SOT_THT:TO-220-3_Vertical" H 3900 5925 50  0001 C CIN
@@
 P 3900 6050
 AR Path="/5EBF8C87" Ref="#PWR?"  Part="1"
-AR Path="/5EBC5EC2/5EBF8C87" Ref="#PWR?"  Part="1"
-F 0 "#PWR?" H 3900 5800 50  0001 C CNN
+AR Path="/5EBC5EC2/5EBF8C87" Ref="#PWR040"  Part="1"
+F 0 "#PWR040" H 3900 5800 50  0001 C CNN
 F 1 "GND" H 3905 5877 50  0000 C CNN
 F 2 "" H 3900 6050 50  0001 C CNN
@@
 P 4300 5900
 AR Path="/5EBF8C8E" Ref="C?"  Part="1"
-AR Path="/5EBC5EC2/5EBF8C8E" Ref="C?"  Part="1"
-F 0 "C?" H 4418 5946 50  0000 L CNN
+AR Path="/5EBC5EC2/5EBF8C8E" Ref="C8"  Part="1"
+F 0 "C8" H 4418 5946 50  0000 L CNN
 F 1 "25uf" H 4418 5855 50  0000 L CNN
 F 2 "Capacitor_THT:CP_Radial_Tantal_D5.0mm_P5.00mm" H 4338 5750 50  0001 C CNN
@@
 P 3550 5900
 AR Path="/5EBF8C94" Ref="C?"  Part="1"
-AR Path="/5EBC5EC2/5EBF8C94" Ref="C?"  Part="1"
-F 0 "C?" H 3665 5946 50  0000 L CNN
+AR Path="/5EBC5EC2/5EBF8C94" Ref="C7"  Part="1"
+F 0 "C7" H 3665 5946 50  0000 L CNN
 F 1 "0.1uf" H 3665 5855 50  0000 L CNN
 F 2 "Capacitor_THT:CP_Radial_Tantal_D5.0mm_P5.00mm" H 3588 5750 50  0001 C CNN
@@
 P 3550 6200
 AR Path="/5EBF8CA0" Ref="#PWR?"  Part="1"
-AR Path="/5EBC5EC2/5EBF8CA0" Ref="#PWR?"  Part="1"
-F 0 "#PWR?" H 3550 5950 50  0001 C CNN
+AR Path="/5EBC5EC2/5EBF8CA0" Ref="#PWR039"  Part="1"
+F 0 "#PWR039" H 3550 5950 50  0001 C CNN
 F 1 "GND" H 3555 6027 50  0000 C CNN
 F 2 "" H 3550 6200 50  0001 C CNN
@@
 P 4300 6200
 AR Path="/5EBF8CA6" Ref="#PWR?"  Part="1"
-AR Path="/5EBC5EC2/5EBF8CA6" Ref="#PWR?"  Part="1"
-F 0 "#PWR?" H 4300 5950 50  0001 C CNN
+AR Path="/5EBC5EC2/5EBF8CA6" Ref="#PWR042"  Part="1"
+F 0 "#PWR042" H 4300 5950 50  0001 C CNN
 F 1 "GND" H 4305 6027 50  0000 C CNN
 F 2 "" H 4300 6200 50  0001 C CNN
@@
 	2900 5650 3550 5650
 $Comp
-L power:+5V #PWR?
+L power:+5V #PWR041
 U 1 1 5EBFB6DE
 P 4300 5700
-F 0 "#PWR?" H 4300 5550 50  0001 C CNN
+F 0 "#PWR041" H 4300 5550 50  0001 C CNN
 F 1 "+5V" H 4315 5873 50  0000 C CNN
 F 2 "" H 4300 5700 50  0001 C CNN
@@
 $EndComp
 $Comp
-L power:+3.3V #PWR?
+L power:+3.3V #PWR038
 U 1 1 5EBFBAE2
 P 2900 5650
-F 0 "#PWR?" H 2900 5500 50  0001 C CNN
+F 0 "#PWR038" H 2900 5500 50  0001 C CNN
 F 1 "+3.3V" H 2915 5823 50  0000 C CNN
 F 2 "" H 2900 5650 50  0001 C CNN
@@
 $EndComp
 $Comp
-L power:+7.5V #PWR?
+L power:+7.5V #PWR043
 U 1 1 5EBFEB12
 P 7500 3400
-F 0 "#PWR?" H 7500 3250 50  0001 C CNN
+F 0 "#PWR043" H 7500 3250 50  0001 C CNN
 F 1 "+7.5V" H 7515 3573 50  0000 C CNN
 F 2 "" H 7500 3400 50  0001 C CNN
@@
 $EndComp
 $Comp
-L Device:R R?
+L Device:R R9
 U 1 1 5EBFF08E
 P 7500 3600
-F 0 "R?" H 7570 3646 50  0000 L CNN
+F 0 "R9" H 7570 3646 50  0000 L CNN
 F 1 "R" H 7570 3555 50  0000 L CNN
 F 2 "" V 7430 3600 50  0001 C CNN
@@
 $EndComp
 $Comp
-L Device:R R?
+L Device:R R10
 U 1 1 5EBFFC02
 P 7500 3900
-F 0 "R?" H 7570 3946 50  0000 L CNN
+F 0 "R10" H 7570 3946 50  0000 L CNN
 F 1 "R" H 7570 3855 50  0000 L CNN
 F 2 "" V 7430 3900 50  0001 C CNN
@@
 $EndComp
 $Comp
-L power:GND #PWR?
+L power:GND #PWR044
 U 1 1 5EC00A08
 P 7500 4050
-F 0 "#PWR?" H 7500 3800 50  0001 C CNN
+F 0 "#PWR044" H 7500 3800 50  0001 C CNN
 F 1 "GND" H 7505 3877 50  0000 C CNN
 F 2 "" H 7500 4050 50  0001 C CNN
