File: CameraTriggerR2PCB/Power.sch (KiCad schematic (older format))
At the start: 16 parts, among them J3 +5V Always on, J4 Ext power switch, J5 Power, SW1 AS11CB, U3 LM7805_TO220

Commit message: Add files via upload
Adding XLR connector
Parts:
- added C7: 0.1uf, Capacitor_THT:CP_Radial_Tantal_D5.0mm_P5.00mm, symbol Device:C
- added C8: 25uf, Capacitor_THT:CP_Radial_Tantal_D5.0mm_P5.00mm, symbol Device:CP
- added R10, R9: R, symbol Device:R
- added U4: LM7803_TO220, Package_TO_SOT_THT:TO-220-3_Vertical, symbol Regulator_Linear:LM7805_TO220
Connections:
- net labels added: +3.3V, V_bat_monitor
- wire segments 44 -> 56
