File: CameraTriggerR2PCB/PushButtons.sch (KiCad schematic (older format))
At the start: 8 parts, among them J10 Trig, J11 Arm, SW2 SW_Trigger, SW3 SW_Arm, SW4 SW_Poll

Commit message: Add files via upload
Changes from 5/17 Zoom sensor
Changed lines of the file:
@@
 	3900 2600 3900 2750
-Wire Wire Line
-	4200 4250 4300 4250
 Wire Wire Line
 	3550 4000 3550 4300
@@
 Wire Wire Line
 	3600 2500 3800 2500
-Wire Wire Line
-	3800 2250 4200 2250
 Wire Wire Line
 	3800 2250 3800 2500
@@
 Connection ~ 4350 3000
 Wire Wire Line
-	4350 3000 4500 3000
-Wire Wire Line
 	4150 3400 4150 3650
 Wire Wire Line
@@
 	3650 2750 3900 2750
 Connection ~ 3900 2750
-Text HLabel 4200 2250 2    50   Input ~ 0
+Text HLabel 5950 2350 2    50   Input ~ 0
 PbTrigIn
-Text HLabel 4500 3000 2    50   Input ~ 0
+Text HLabel 5950 3000 2    50   Input ~ 0
 ArmIn
-Text HLabel 4300 4250 2    50   Input ~ 0
+Text HLabel 5950 4200 2    50   Input ~ 0
 Poll
+Wire Wire Line
+	5900 2250 5900 2350
+Wire Wire Line
+	5900 2350 5950 2350
+Wire Wire Line
+	3800 2250 5900 2250
+Wire Wire Line
+	4350 3000 5950 3000
+Wire Wire Line
+	5850 4250 5850 4200
+Wire Wire Line
+	5850 4200 5950 4200
+Wire Wire Line
+	4200 4250 5850 4250
 $EndSCHEMATC
