File: CameraTriggerR2PCB/RFM95.sch (KiCad schematic (older format))
At the start: 3 parts

Commit message: Add files via upload
Changes from 5/17 Zoom sensor
Parts:
- gave numbers to parts that had none: 3
Changed lines of the file:
@@
 $EndDescr
 $Comp
-L power:+3.3V #PWR?
+L power:+3.3V #PWR047
 U 1 1 5EBC2ECD
 P 4350 2400
-F 0 "#PWR?" H 4350 2250 50  0001 C CNN
+F 0 "#PWR047" H 4350 2250 50  0001 C CNN
 F 1 "+3.3V" H 4365 2573 50  0000 C CNN
 F 2 "" H 4350 2400 50  0001 C CNN
@@
 	4350 3050 4350 2500
 $Comp
-L Device:C C?
+L Device:C C9
 U 1 1 5EBC3B26
 P 4800 2650
-F 0 "C?" H 4915 2696 50  0000 L CNN
+F 0 "C9" H 4915 2696 50  0000 L CNN
 F 1 "10nf" H 4915 2605 50  0000 L CNN
 F 2 "" H 4838 2500 50  0001 C CNN
@@
 $EndComp
 $Comp
-L power:GND #PWR?
+L power:GND #PWR049
 U 1 1 5EBC3E8B
 P 4800 2800
-F 0 "#PWR?" H 4800 2550 50  0001 C CNN
+F 0 "#PWR049" H 4800 2550 50  0001 C CNN
 F 1 "GND" H 4805 2627 50  0000 C CNN
 F 2 "" H 4800 2800 50  0001 C CNN
@@
 $EndComp
 $Comp
-L power:GND #PWR?
+L power:GND #PWR048
 U 1 1 5EBC427B
 P 4450 4450
-F 0 "#PWR?" H 4450 4200 50  0001 C CNN
+F 0 "#PWR048" H 4450 4200 50  0001 C CNN
 F 1 "GND" H 4455 4277 50  0000 C CNN
 F 2 "" H 4450 4450 50  0001 C CNN
@@
 	4250 4150 4350 4150
 $Comp
-L RF_Module:RFM95W-915S2 U?
+L RF_Module:RFM95W-915S2 U5
 U 1 1 5EBC207D
 P 4350 3550
-F 0 "U?" H 4350 4231 50  0000 C CNN
+F 0 "U5" H 4350 4231 50  0000 C CNN
 F 1 "RFM95W-915S2" H 4350 4140 50  0000 C CNN
 F 2 "" H 1050 5200 50  0001 C CNN
@@
 NoConn ~ 4850 3450
 $Comp
-L Connector:Conn_Coaxial J?
+L Connector:Conn_Coaxial J14
 U 1 1 5EBC6410
 P 5050 3250
-F 0 "J?" H 5150 3225 50  0000 L CNN
+F 0 "J14" H 5150 3225 50  0000 L CNN
 F 1 "Conn_Coaxial" H 5150 3134 50  0000 L CNN
 F 2 "" H 5050 3250 50  0001 C CNN
@@
 $EndComp
 $Comp
-L power:GND #PWR?
+L power:GND #PWR050
 U 1 1 5EBC6AD9
 P 5050 3450
-F 0 "#PWR?" H 5050 3200 50  0001 C CNN
+F 0 "#PWR050" H 5050 3200 50  0001 C CNN
 F 1 "GND" H 5055 3277 50  0000 C CNN
 F 2 "" H 5050 3450 50  0001 C CNN
@@
 Text Notes 6250 3050 0    50   ~ 0
 Based on Feather M0 LoRa Adafruit  3178
+Connection ~ 3850 3250
+Connection ~ 4850 3950
+Connection ~ 3850 3750
+Connection ~ 3850 3550
+Connection ~ 3850 3450
+Connection ~ 3850 3350
 $EndSCHEMATC
