File: CameraTriggerR2PCB/WiFi_BT.sch (KiCad schematic (older format))
At the start: 10 parts, among them IC4 NINA-W102

Commit message: Add files via upload
Changes from 5/17 Zoom sensor
Parts:
- gave numbers to parts that had none: 9
Connections:
- net labels removed: BT_WIFI_CS, BT_WIFI_MISO, BT_WIFI_MOSI, BT_WIFI_SCK
- no-connect marks 0 -> 14
Changed lines of the file:
@@
 $EndComp
 $Comp
-L power:GND #PWR?
+L power:GND #PWR058
 U 1 1 5EB641E1
 P 8250 5100
-F 0 "#PWR?" H 8250 4850 50  0001 C CNN
+F 0 "#PWR058" H 8250 4850 50  0001 C CNN
 F 1 "GND" H 8255 4927 50  0000 C CNN
 F 2 "" H 8250 5100 50  0001 C CNN
@@
 	8250 4750 8250 5100
 $Comp
-L power:GND #PWR?
+L power:GND #PWR056
 U 1 1 5EB65974
 P 8200 2600
-F 0 "#PWR?" H 8200 2350 50  0001 C CNN
+F 0 "#PWR056" H 8200 2350 50  0001 C CNN
 F 1 "GND" H 8205 2427 50  0000 C CNN
 F 2 "" H 8200 2600 50  0001 C CNN
@@
 	8200 2550 8200 2600
 $Comp
-L power:GND #PWR?
+L power:GND #PWR059
 U 1 1 5EB6622F
 P 8300 2950
-F 0 "#PWR?" H 8300 2700 50  0001 C CNN
+F 0 "#PWR059" H 8300 2700 50  0001 C CNN
 F 1 "GND" H 8305 2777 50  0000 C CNN
 F 2 "" H 8300 2950 50  0001 C CNN
@@
 	7500 2950 8300 2950
 $Comp
-L power:GND #PWR?
+L power:GND #PWR051
 U 1 1 5EB66F6E
 P 2700 3800
-F 0 "#PWR?" H 2700 3550 50  0001 C CNN
+F 0 "#PWR051" H 2700 3550 50  0001 C CNN
 F 1 "GND" H 2705 3627 50  0000 C CNN
 F 2 "" H 2700 3800 50  0001 C CNN
@@
 	3500 3550 3150 3550
 $Comp
-L power:+3.3V #PWR?
+L power:+3.3V #PWR053
 U 1 1 5EB67963
 P 2750 3150
-F 0 "#PWR?" H 2750 3000 50  0001 C CNN
+F 0 "#PWR053" H 2750 3000 50  0001 C CNN
 F 1 "+3.3V" H 2765 3323 50  0000 C CNN
 F 2 "" H 2750 3150 50  0001 C CNN
@@
 	3000 4450 3200 4450
 $Comp
-L Connector:Conn_01x05_Male J?
+L Connector:Conn_01x05_Male J16
 U 1 1 5EB9F685
 P 9550 3400
-F 0 "J?" H 9658 3781 50  0000 C CNN
+F 0 "J16" H 9658 3781 50  0000 C CNN
 F 1 "JTAG" H 9658 3690 50  0000 C CNN
 F 2 "" H 9550 3400 50  0001 C CNN
@@
 Reset_N
 $Comp
-L power:GND #PWR?
+L power:GND #PWR052
 U 1 1 5EBA8D2B
 P 2750 2600
-F 0 "#PWR?" H 2750 2350 50  0001 C CNN
+F 0 "#PWR052" H 2750 2350 50  0001 C CNN
 F 1 "GND" H 2755 2427 50  0000 C CNN
 F 2 "" H 2750 2600 50  0001 C CNN
@@
 $EndComp
 $Comp
-L Switch:SW_Push SW?
+L Switch:SW_Push SW5
 U 1 1 5EBAFBBA
 P 8050 1300
-F 0 "SW?" H 8050 1585 50  0000 C CNN
+F 0 "SW5" H 8050 1585 50  0000 C CNN
 F 1 "SW_Push" H 8050 1494 50  0000 C CNN
 F 2 "" H 8050 1500 50  0001 C CNN
@@
 $EndComp
 $Comp
-L power:GND #PWR?
+L power:GND #PWR057
 U 1 1 5EBAFBC0
 P 8250 1400
-F 0 "#PWR?" H 8250 1150 50  0001 C CNN
+F 0 "#PWR057" H 8250 1150 50  0001 C CNN
 F 1 "GND" H 8255 1227 50  0000 C CNN
 F 2 "" H 8250 1400 50  0001 C CNN
@@
 	8250 1300 8250 1400
 $Comp
-L Device:R R?
+L Device:R R13
 U 1 1 5EBAFBC7
 P 7600 1150
-F 0 "R?" H 7670 1196 50  0000 L CNN
+F 0 "R13" H 7670 1196 50  0000 L CNN
 F 1 "10K" H 7670 1105 50  0000 L CNN
 F 2 "" V 7530 1150 50  0001 C CNN
@@
 $EndComp
 $Comp
-L power:+3.3V #PWR?
+L power:+3.3V #PWR055
 U 1 1 5EBAFBCE
 P 7600 950
-F 0 "#PWR?" H 7600 800 50  0001 C CNN
+F 0 "#PWR055" H 7600 800 50  0001 C CNN
 F 1 "+3.3V" H 7615 1123 50  0000 C CNN
 F 2 "" H 7600 950 50  0001 C CNN
@@
 	2750 2500 2750 2600
 $Comp
-L Device:C C?
+L Device:C C11
 U 1 1 5EBB2A66
 P 7250 1450
-F 0 "C?" H 7365 1496 50  0000 L CNN
+F 0 "C11" H 7365 1496 50  0000 L CNN
 F 1 "10nF" H 7365 1405 50  0000 L CNN
 F 2 "" H 7288 1300 50  0001 C CNN
@@
 $EndComp
 $Comp
-L power:GND #PWR?
+L power:GND #PWR054
 U 1 1 5EBB2DE1
 P 7250 1600
-F 0 "#PWR?" H 7250 1350 50  0001 C CNN
+F 0 "#PWR054" H 7250 1350 50  0001 C CNN
 F 1 "GND" H 7255 1427 50  0000 C CNN
 F 2 "" H 7250 1600 50  0001 C CNN
@@
 	7600 1300 7850 1300
 $Comp
-L Device:C C?
+L Device:C C10
 U 1 1 5EBC985D
 P 2300 3450
-F 0 "C?" H 2415 3496 50  0000 L CNN
+F 0 "C10" H 2415 3496 50  0000 L CNN
 F 1 "10nF" H 2415 3405 50  0000 L CNN
 F 2 "" H 2338 3300 50  0001 C CNN
@@
 AR Path="/5E9FE63A/5EBD38BF" Ref="#PWR?"  Part="1"
 AR Path="/5EA0B5A0/5EBD38BF" Ref="#PWR?"  Part="1"
-AR Path="/5EBC729C/5EBD38BF" Ref="#PWR?"  Part="1"
-F 0 "#PWR?" H 10800 1650 50  0001 C CNN
+AR Path="/5EBC729C/5EBD38BF" Ref="#PWR062"  Part="1"
+F 0 "#PWR062" H 10800 1650 50  0001 C CNN
 F 1 "GND" H 10805 1727 50  0000 C CNN
 F 2 "" H 10800 1900 50  0001 C CNN
@@
 AR Path="/5E9FE63A/5EBD38C8" Ref="10K?"  Part="1"
 AR Path="/5EA0B5A0/5EBD38C8" Ref="10K?"  Part="1"
-AR Path="/5EBC729C/5EBD38C8" Ref="10K?"  Part="1"
-F 0 "10K?" H 10170 1396 50  0000 L CNN
+AR Path="/5EBC729C/5EBD38C8" Ref="10K1"  Part="1"
+F 0 "10K1" H 10170 1396 50  0000 L CNN
 F 1 "R" H 10170 1305 50  0000 L CNN
 F 2 "" V 10030 1350 50  0001 C CNN
@@
 AR Path="/5E9FE63A/5EBD38CE" Ref="#PWR?"  Part="1"
 AR Path="/5EA0B5A0/5EBD38CE" Ref="#PWR?"  Part="1"
-AR Path="/5EBC729C/5EBD38CE" Ref="#PWR?"  Part="1"
-F 0 "#PWR?" H 10100 950 50  0001 C CNN
+AR Path="/5EBC729C/5EBD38CE" Ref="#PWR060"  Part="1"
+F 0 "#PWR060" H 10100 950 50  0001 C CNN
 F 1 "+3.3V" H 10115 1273 50  0000 C CNN
 F 2 "" H 10100 1100 50  0001 C CNN
@@
 AR Path="/5E9FE63A/5EBD38D8" Ref="10K?"  Part="1"
 AR Path="/5EA0B5A0/5EBD38D8" Ref="10K?"  Part="1"
-AR Path="/5EBC729C/5EBD38D8" Ref="10K?"  Part="1"
-F 0 "10K?" H 10170 1846 50  0000 L CNN
+AR Path="/5EBC729C/5EBD38D8" Ref="10K2"  Part="1"
+F 0 "10K2" H 10170 1846 50  0000 L CNN
 F 1 "R" H 10170 1755 50  0000 L CNN
 F 2 "" V 10030 1800 50  0001 C CNN
@@
 AR Path="/5E9FE63A/5EBD38DE" Ref="#PWR?"  Part="1"
 AR Path="/5EA0B5A0/5EBD38DE" Ref="#PWR?"  Part="1"
-AR Path="/5EBC729C/5EBD38DE" Ref="#PWR?"  Part="1"
-F 0 "#PWR?" H 10100 1900 50  0001 C CNN
+AR Path="/5EBC729C/5EBD38DE" Ref="#PWR061"  Part="1"
+F 0 "#PWR061" H 10100 1900 50  0001 C CNN
 F 1 "+3.3V" H 10115 2223 50  0000 C CNN
 F 2 "" H 10100 2050 50  0001 C CNN
@@
 	10100 1950 10100 2050
 $Comp
-L Switch:SW_DIP_x02 SW?
+L Switch:SW_DIP_x02 SW6
 U 1 1 5EBD38E5
 P 10500 1650
-F 0 "SW?" H 10500 2017 50  0000 C CNN
+F 0 "SW6" H 10500 2017 50  0000 C CNN
 F 1 "SW_DIP_x02" H 10500 1926 50  0000 C CNN
 F 2 "" H 10500 1650 50  0001 C CNN
@@
 	7500 2650 8800 2650
 $Comp
-L Connector:Conn_01x05_Male J?
+L Connector:Conn_01x05_Male J15
 U 1 1 5EBDB92E
 P 3200 5000
-F 0 "J?" V 3262 5244 50  0000 L CNN
+F 0 "J15" V 3262 5244 50  0000 L CNN
 F 1 "Serial/USB" V 3353 5244 50  0000 L CNN
 F 2 "" H 3200 5000 50  0001 C CNN
@@
 Text Notes 5550 5550 0    50   ~ 0
 Todo - put crystal on\nBreak MISO/MISI/SCK/CS lines  (goes to MCU)
-Text HLabel 4350 6050 0    50   Input ~ 0
-BT_WIFI_MISO
-Text HLabel 4350 6250 0    50   Input ~ 0
-BT_WIFI_MOSI
-Text HLabel 4350 6400 0    50   Input ~ 0
-BT_WIFI_CS
-Text HLabel 4300 6500 0    50   Input ~ 0
-BT_WIFI_SCK
+NoConn ~ 3500 2450
+NoConn ~ 3500 2550
+NoConn ~ 3500 2650
+NoConn ~ 3500 2750
+NoConn ~ 3500 2850
+NoConn ~ 3500 3050
+NoConn ~ 3500 3150
+NoConn ~ 3500 3450
+NoConn ~ 3500 3650
+NoConn ~ 3500 3850
+NoConn ~ 3500 3950
+NoConn ~ 3500 4050
+NoConn ~ 3500 4150
+NoConn ~ 3500 4750
+Connection ~ 3500 2950
+Connection ~ 3500 3250
+Connection ~ 3500 3350
+Connection ~ 3500 3550
+Connection ~ 3500 3750
+Connection ~ 3500 4250
+Connection ~ 3500 4350
+Connection ~ 3500 4450
+Connection ~ 3500 4550
+Connection ~ 3500 4650
 $EndSCHEMATC

Commit message: Add files via upload
Updates from last few sessions
Parts:
- added X?: SG-3030CM, Oscillator:Oscillator_SMD_SeikoEpson_SG3030CM, symbol Oscillator:SG-3030CM
Connections:
- net labels added: NINA_ACK, NINA_CTS_SCK, NINA_GPIO0, NINA_MISO, NINA_MOSI, NINA_RESETN, NINA_RTS_CS, NINA_RX, NINA_TX
- net labels removed: BT_WIFI_CTS, BT_WIFI_RTS, BT_WIFI_RX, BT_WIFI_TX, Reset_N
- wire segments 93 -> 98
- no-connect marks 14 -> 11
Changed lines of the file:
@@
 EESchema Schematic File Version 4
-LIBS:CameraTrigger-cache
 EELAYER 30 0
 EELAYER END
 $Descr A4 11693 8268
 encoding utf-8
-Sheet 8 9
+Sheet 1 1
 Title ""
 Date ""
@@
 	3150 3550 2700 3550
 Text HLabel 3000 4550 0    50   Input ~ 0
-BT_WIFI_TX
+NINA_TX
 Text HLabel 3000 4650 0    50   Input ~ 0
-BT_WIFI_RX
+NINA_RX
 Text HLabel 3000 4350 0    50   Input ~ 0
-BT_WIFI_RTS
+NINA_RTS_CS
 Text HLabel 3000 4450 0    50   Input ~ 0
-BT_WIFI_CTS
+NINA_CTS_SCK
 Wire Wire Line
 	3000 4350 3100 4350
@@
 	9450 3600 9550 3600
 Text HLabel 2900 4250 0    50   Input ~ 0
-Reset_N
+NINA_RESETN
 $Comp
 L power:GND #PWR052
@@
 AR Path="/5EA0B5A0/5EBD38BF" Ref="#PWR?"  Part="1"
 AR Path="/5EBC729C/5EBD38BF" Ref="#PWR062"  Part="1"
+AR Path="/5EBD38BF" Ref="#PWR062"  Part="1"
 F 0 "#PWR062" H 10800 1650 50  0001 C CNN
 F 1 "GND" H 10805 1727 50  0000 C CNN
@@
 AR Path="/5EA0B5A0/5EBD38C8" Ref="10K?"  Part="1"
 AR Path="/5EBC729C/5EBD38C8" Ref="10K1"  Part="1"
+AR Path="/5EBD38C8" Ref="10K1"  Part="1"
 F 0 "10K1" H 10170 1396 50  0000 L CNN
 F 1 "R" H 10170 1305 50  0000 L CNN
@@
 AR Path="/5EA0B5A0/5EBD38CE" Ref="#PWR?"  Part="1"
 AR Path="/5EBC729C/5EBD38CE" Ref="#PWR060"  Part="1"
+AR Path="/5EBD38CE" Ref="#PWR060"  Part="1"
 F 0 "#PWR060" H 10100 950 50  0001 C CNN
 F 1 "+3.3V" H 10115 1273 50  0000 C CNN
@@
 AR Path="/5EA0B5A0/5EBD38D8" Ref="10K?"  Part="1"
 AR Path="/5EBC729C/5EBD38D8" Ref="10K2"  Part="1"
+AR Path="/5EBD38D8" Ref="10K2"  Part="1"
 F 0 "10K2" H 10170 1846 50  0000 L CNN
 F 1 "R" H 10170 1755 50  0000 L CNN
@@
 AR Path="/5EA0B5A0/5EBD38DE" Ref="#PWR?"  Part="1"
 AR Path="/5EBC729C/5EBD38DE" Ref="#PWR061"  Part="1"
+AR Path="/5EBD38DE" Ref="#PWR061"  Part="1"
 F 0 "#PWR061" H 10100 1900 50  0001 C CNN
 F 1 "+3.3V" H 10115 2223 50  0000 C CNN
@@
 Text Notes 5550 5550 0    50   ~ 0
 Todo - put crystal on\nBreak MISO/MISI/SCK/CS lines  (goes to MCU)
-NoConn ~ 3500 2450
 NoConn ~ 3500 2550
 NoConn ~ 3500 2650
 NoConn ~ 3500 2750
-NoConn ~ 3500 2850
-NoConn ~ 3500 3050
 NoConn ~ 3500 3150
 NoConn ~ 3500 3450
@@
 NoConn ~ 3500 4150
 NoConn ~ 3500 4750
-Connection ~ 3500 2950
-Connection ~ 3500 3250
-Connection ~ 3500 3350
-Connection ~ 3500 3550
-Connection ~ 3500 3750
-Connection ~ 3500 4250
-Connection ~ 3500 4350
-Connection ~ 3500 4450
-Connection ~ 3500 4550
-Connection ~ 3500 4650
+$Comp
+L Oscillator:SG-3030CM X?
+U 1 1 5EC5D6A2
+P 2050 2000
+F 0 "X?" H 1821 2046 50  0000 R CNN
+F 1 "SG-3030CM" H 1821 1955 50  0000 R CNN
+F 2 "Oscillator:Oscillator_SMD_SeikoEpson_SG3030CM" H 2050 1650 50  0001 C CNN
+F 3 "https://support.epson.biz/td/api/doc_check.php?mode=dl&lang=en&Parts=SG-3030CM" H 1950 2000 50  0001 C CNN
+	1    2050 2000
+	1    0    0    -1
+$EndComp
+Wire Wire Line
+	2350 2000 3250 2000
+Wire Wire Line
+	3250 2000 3250 2850
+Wire Wire Line
+	3250 2850 3500 2850
+Connection ~ 3500 2850
+Wire Wire Line
+	3500 2850 3550 2850
+$Comp
+L power:GND #PWR?
+U 1 1 5EC67323
+P 2050 2300
+F 0 "#PWR?" H 2050 2050 50  0001 C CNN
+F 1 "GND" H 2055 2127 50  0000 C CNN
+F 2 "" H 2050 2300 50  0001 C CNN
+F 3 "" H 2050 2300 50  0001 C CNN
+	1    2050 2300
+	1    0    0    -1
+$EndComp
+$Comp
+L power:+3.3V #PWR?
+U 1 1 5EC67736
+P 1950 1700
+F 0 "#PWR?" H 1950 1550 50  0001 C CNN
+F 1 "+3.3V" H 1965 1873 50  0000 C CNN
+F 2 "" H 1950 1700 50  0001 C CNN
+F 3 "" H 1950 1700 50  0001 C CNN
+	1    1950 1700
+	1    0    0    -1
+$EndComp
+Wire Wire Line
+	1950 1700 2150 1700
+Connection ~ 1950 1700
+Text HLabel 3450 3050 0    50   Input ~ 0
+NINA_ACK
+Text HLabel 3700 1700 0    50   Input ~ 0
+NINA_GPIO0
+Text HLabel 2100 4300 0    50   Input ~ 0
+NINA_MISO
+Text HLabel 3500 2450 0    50   Input ~ 0
+NINA_MOSI
 $EndSCHEMATC
