File: CameraTriggerR2PCB/CameraTriggerSensorNodeOnly.sch (KiCad schematic (older format))
At the start: 43 parts, among them IC1 3178, J1 Power, J13 Serial, J14 Ext power switch, J2 Qwiic_Connector, J3 Aux out, J4 HighLowIn, J5 Laser, J6 Sensor, Q1 PN2222A, SW1 AS11CB, SW3 SW_Poll, U1 LM7805_TO220

Commit message: Add files via upload
Rdo SCK SDL to correct pins
Connections:
- no-connect marks 19 -> 20
Changed lines of the file:
@@
 Text Label 5650 4450 2    50   ~ 0
 SDA
-Wire Wire Line
-	5400 4350 5650 4350
-Wire Wire Line
-	5400 4450 5650 4450
 Text GLabel 5850 4250 2    50   Input ~ 0
 SensorIn
-NoConn ~ 5650 4350
-NoConn ~ 5650 4450
 Text GLabel 5850 4150 2    50   Input ~ 0
 ArmInd
@@
 Wire Wire Line
 	2150 5250 2450 5250
-Text GLabel 3300 4150 0    50   Input ~ 0
+Text GLabel 5850 4350 2    50   Input ~ 0
 SCL_qwiic
-Text GLabel 3300 4250 0    50   Input ~ 0
+Text GLabel 5850 4450 2    50   Input ~ 0
 SDA_qwiic
 Wire Wire Line
 	3300 3950 4000 3950
-Wire Wire Line
-	3300 4250 4000 4250
-Wire Wire Line
-	3300 4150 4000 4150
 NoConn ~ 3300 3950
 $Comp
@@
 Text GLabel 3300 4050 0    50   Input ~ 0
 Threshold
+Wire Wire Line
+	5400 4350 5850 4350
+Wire Wire Line
+	5400 4450 5850 4450
+Wire Wire Line
+	3800 4150 4000 4150
+Wire Wire Line
+	3800 4250 4000 4250
+NoConn ~ 3800 4150
+NoConn ~ 3800 4250
+NoConn ~ 5500 3100
 $EndSCHEMATC

Commit message: Add files via upload
Adding XLR connector
Parts:
- added J7: XLR5, Jack_XLR_Neutrik_NC5FAV-DA_Vertical, symbol Connector:XLR5
- added J8: (no value), Connector_PinHeader_2.54mm:PinHeader_1x03_P2.54mm_Vertical, symbol Connector:Conn_01x03_Male
- added Q2: KSC1815YTA, Package_TO_SOT_THT:TO-92L_Inline_Wide, symbol Transistor_BJT:2SC1815
- added R2, R6: 1K, Resistor_THT:R_Axial_DIN0207_L6.3mm_D2.5mm_P7.62mm_Horizontal, symbol Device:R
- added SW2: SW_Arm, Button_Switch_THT:KSA_Tactile_SPST, symbol Switch:SW_Push
- H2, H3: value MountingHole_Pad -> (none)
- Q1: footprint Package_TO_SOT_THT:TO-92_Inline -> Package_TO_SOT_THT:TO-92L_HandSolder
- TP1: value TestPoint -> Gnd
Connections:
- net labels added: ArmIn, HighLow, Laser, LowHigh
- wire segments 151 -> 146
- no-connect marks 20 -> 19
Other:
- moved on the sheet: BZ1, C3, C4, C5, C6, D2, GND1, H2, H3, H4, R5, SW3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

Commit message: Add files via upload
Production version
Parts:
- removed J8: (no value), Connector_PinHeader_2.54mm:PinHeader_1x03_P2.54mm_Vertical, symbol Connector:Conn_01x03_Male
- added SW4: SW_SPDT, Button_Switch_THT:SW_Slide_1P2T_CK_OS102011MS2Q, symbol Switch:SW_SPDT
- J7: footprint Jack_XLR_Neutrik_NC5FAV-DA_Vertical -> SamacSys_Parts:Jack_XLR_Neutrik_NC5MBH_Horizontal
Changed lines of the file:
@@
 F 0 "J7" H 3350 5715 50  0000 C CNN
 F 1 "XLR5" H 3350 5624 50  0000 C CNN
-F 2 "Jack_XLR_Neutrik_NC5FAV-DA_Vertical" H 3350 5350 50  0001 C CNN
+F 2 "SamacSys_Parts:Jack_XLR_Neutrik_NC5MBH_Horizontal" H 3350 5350 50  0001 C CNN
 F 3 " ~" H 3350 5350 50  0001 C CNN
 	1    3350 5350
@@
 	-1   0    0    1
 $EndComp
-$Comp
-L Connector:Conn_01x03_Male J8
-U 1 1 5ED3C6BA
-P 4800 5950
-F 0 "J8" H 4908 6231 50  0000 C CNN
-F 1 " " H 4908 6140 50  0000 C CNN
-F 2 "Connector_PinHeader_2.54mm:PinHeader_1x03_P2.54mm_Vertical" H 4800 5950 50  0001 C CNN
-F 3 "~" H 4800 5950 50  0001 C CNN
-	1    4800 5950
-	-1   0    0    1
-$EndComp
 Wire Wire Line
 	3650 5950 3650 5450
@@
 Wire Wire Line
 	5700 6800 5800 6800
-Text GLabel 4600 5850 0    50   Input ~ 0
+Text GLabel 5000 5850 2    50   Input ~ 0
 AuxIn
-Text GLabel 4600 6050 0    50   Input ~ 0
+Text GLabel 5000 6050 2    50   Input ~ 0
 SensorIn
 Wire Wire Line
 	3650 5950 4600 5950
-Text Label 4900 5850 0    50   ~ 0
+Text Label 5350 5850 0    50   ~ 0
 HighLow
-Text Label 4900 6050 0    50   ~ 0
+Text Label 5350 6050 0    50   ~ 0
 LowHigh
-Connection ~ 4600 6050
+$Comp
+L Switch:SW_SPDT SW4
+U 1 1 5ED58B25
+P 4800 5950
+F 0 "SW4" H 4800 6235 50  0000 C CNN
+F 1 "SW_SPDT" H 4800 6144 50  0000 C CNN
+F 2 "Button_Switch_THT:SW_Slide_1P2T_CK_OS102011MS2Q" H 4800 5950 50  0001 C CNN
+F 3 "~" H 4800 5950 50  0001 C CNN
+	1    4800 5950
+	1    0    0    -1
+$EndComp
 $EndSCHEMATC

Commit message: Add files via upload
Added comment to schematic for XLR connector (male).
Parts:
- J7: value XLR5 -> XLR5 Male
Changed lines of the file:
@@
 P 3350 5350
 F 0 "J7" H 3350 5715 50  0000 C CNN
-F 1 "XLR5" H 3350 5624 50  0000 C CNN
+F 1 "XLR5 Male" H 3350 5624 50  0000 C CNN
 F 2 "SamacSys_Parts:Jack_XLR_Neutrik_NC5MBH_Horizontal" H 3350 5350 50  0001 C CNN
 F 3 " ~" H 3350 5350 50  0001 C CNN
